File: pcb.brd (EAGLE design)
At the start: 121 x 83 mm, 22 parts

Commit message: Minor enhancements
Parts:
- moved S1 3.00 mm to (12.0, 37.0)
Routing:
- net N$31: track 117.1 -> 123.4 mm
- net N$30: track 153.0 -> 156.3 mm
- net N$36: track 109.4 -> 112.5 mm
- net N$26: track 39.9 -> 42.9 mm
- net N$28: track 39.4 -> 42.3 mm
- net N$1: track 121.1 -> 122.2 mm
Changed lines of the file:
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@@
 <element name="U$8" library="cherrymx" package="CHERRY-MX-DIODE" value="CHERRY-MX-DIODE" x="70" y="51" rot="R90"/>
 <element name="U$9" library="cherrymx" package="CHERRY-MX-DIODE" value="CHERRY-MX-DIODE" x="89" y="51" rot="R90"/>
-<element name="S1" library="SparkFun-Switches" package="TACTILE_SWITCH_PTH_12MM" value="RESET" x="12" y="40" rot="MR90">
-<attribute name="PROD_ID" value="SWCH-09185" x="12" y="40" size="1.778" layer="28" rot="MR90" display="off"/>
-<attribute name="SF_SKU" value="COM-09190" x="12" y="40" size="1.778" layer="28" rot="MR90" display="off"/>
+<element name="S1" library="SparkFun-Switches" package="TACTILE_SWITCH_PTH_12MM" value="RESET" x="12" y="37" rot="MR90">
+<attribute name="PROD_ID" value="SWCH-09185" x="12" y="37" size="1.778" layer="28" rot="MR90" display="off"/>
+<attribute name="SF_SKU" value="COM-09190" x="12" y="37" size="1.778" layer="28" rot="MR90" display="off"/>
 </element>
 </elements>
@@
 <contactref element="B1" pad="8"/>
 <wire x1="22" y1="13" x2="21" y2="14" width="0.4064" layer="1"/>
-<wire x1="21" y1="14" x2="21" y2="47" width="0.4064" layer="1"/>
-<wire x1="16" y1="52" x2="13" y2="52" width="0.4064" layer="1"/>
+<wire x1="21" y1="14" x2="21" y2="49" width="0.4064" layer="1"/>
+<wire x1="18" y1="52" x2="13" y2="52" width="0.4064" layer="1"/>
 <wire x1="28.7806" y1="13" x2="22" y2="13" width="0.4064" layer="1"/>
-<wire x1="21" y1="47" x2="16" y2="52" width="0.4064" layer="1"/>
+<wire x1="21" y1="49" x2="18" y2="52" width="0.4064" layer="1"/>
 <wire x1="13" y1="52" x2="6.38" y2="60.92" width="0.4064" layer="1"/>
 <wire x1="28.7806" y1="13" x2="28.7806" y2="14.333525" width="0" layer="19" extent="1-1"/>
@@
 <wire x1="47.7806" y1="11.666475" x2="48.46" y2="10.987075" width="0.4064" layer="1"/>
 <wire x1="48.46" y1="10.987075" x2="48.46" y2="9.19" width="0.4064" layer="1"/>
-<wire x1="22" y1="5" x2="20" y2="7" width="0.4064" layer="1"/>
-<wire x1="41" y1="5" x2="22" y2="5" width="0.4064" layer="1"/>
+<wire x1="23" y1="5" x2="20" y2="8" width="0.4064" layer="1"/>
+<wire x1="41" y1="5" x2="23" y2="5" width="0.4064" layer="1"/>
 <wire x1="47.7806" y1="13" x2="43" y2="13" width="0.4064" layer="1"/>
 <wire x1="43" y1="13" x2="43" y2="7" width="0.4064" layer="1"/>
 <wire x1="43" y1="7" x2="41" y2="5" width="0.4064" layer="1"/>
 <contactref element="B1" pad="9"/>
-<wire x1="20" y1="47" x2="16" y2="51" width="0.4064" layer="1"/>
+<wire x1="20" y1="48" x2="17" y2="51" width="0.4064" layer="1"/>
 <wire x1="12" y1="51" x2="6.38" y2="58.38" width="0.4064" layer="1"/>
-<wire x1="20" y1="7" x2="20" y2="47" width="0.4064" layer="1"/>
-<wire x1="16" y1="51" x2="12" y2="51" width="0.4064" layer="1"/>
+<wire x1="20" y1="8" x2="20" y2="48" width="0.4064" layer="1"/>
+<wire x1="17" y1="51" x2="12" y2="51" width="0.4064" layer="1"/>
 </signal>
 <signal name="N$4">
@@
 <wire x1="81" y1="8" x2="81" y2="13" width="0.4064" layer="1"/>
 <contactref element="B1" pad="11"/>
-<wire x1="16" y1="49" x2="18" y2="47" width="0.4064" layer="1"/>
-<wire x1="16" y1="49" x2="10" y2="49" width="0.4064" layer="1"/>
+<wire x1="15" y1="49" x2="18" y2="46" width="0.4064" layer="1"/>
+<wire x1="15" y1="49" x2="10" y2="49" width="0.4064" layer="1"/>
 <wire x1="10" y1="49" x2="6.38" y2="53.3" width="0.4064" layer="1"/>
-<wire x1="18" y1="7" x2="22" y2="3" width="0.4064" layer="1"/>
-<wire x1="22" y1="3" x2="76" y2="3" width="0.4064" layer="1"/>
-<wire x1="18" y1="47" x2="18" y2="7" width="0.4064" layer="1"/>
+<wire x1="18" y1="6" x2="21" y2="3" width="0.4064" layer="1"/>
+<wire x1="21" y1="3" x2="76" y2="3" width="0.4064" layer="1"/>
+<wire x1="18" y1="46" x2="18" y2="6" width="0.4064" layer="1"/>
 <wire x1="76" y1="3" x2="81" y2="8" width="0.4064" layer="1"/>
 <wire x1="85.7806" y1="13" x2="85.7806" y2="14.333525" width="0" layer="19" extent="1-1"/>
@@
 <wire x1="6.38" y1="50.76" x2="6.38" y2="50.62" width="0.4064" layer="1"/>
 <wire x1="6.38" y1="50.62" x2="9" y2="48" width="0.4064" layer="1"/>
-<wire x1="9" y1="48" x2="16" y2="48" width="0.4064" layer="1"/>
-<wire x1="16" y1="48" x2="17" y2="47" width="0.4064" layer="1"/>
-<wire x1="17" y1="47" x2="17" y2="7" width="0.4064" layer="1"/>
-<wire x1="17" y1="7" x2="22" y2="2" width="0.4064" layer="1"/>
-<wire x1="22" y1="2" x2="96" y2="2" width="0.4064" layer="1"/>
+<wire x1="9" y1="48" x2="14" y2="48" width="0.4064" layer="1"/>
+<wire x1="14" y1="48" x2="17" y2="45" width="0.4064" layer="1"/>
+<wire x1="17" y1="45" x2="17" y2="5" width="0.4064" layer="1"/>
+<wire x1="17" y1="5" x2="20" y2="2" width="0.4064" layer="1"/>
+<wire x1="20" y1="2" x2="96" y2="2" width="0.4064" layer="1"/>
 <wire x1="96" y1="2" x2="100" y2="6" width="0.4064" layer="1"/>
 <wire x1="104.7806" y1="13" x2="104.7806" y2="14.333525" width="0" layer="19" extent="1-1"/>
@@
 <wire x1="103.08920625" y1="47.19" x2="106.05140625" y2="44.2278" width="0.4064" layer="16"/>
 <wire x1="106.05140625" y1="44.2278" x2="108.7009375" y2="44.2278" width="0.4064" layer="16"/>
-<wire x1="25" y1="51.46" x2="25" y2="44" width="0.4064" layer="16"/>
-<wire x1="25" y1="51.46" x2="21.62" y2="55.84" width="0.4064" layer="16"/>
-<wire x1="38.81" y1="44" x2="42" y2="47.19" width="0.4064" layer="16"/>
-<wire x1="25" y1="44" x2="38.81" y2="44" width="0.4064" layer="16"/>
+<wire x1="24" y1="55" x2="24" y2="43" width="0.4064" layer="16"/>
+<wire x1="24" y1="43" x2="25" y2="42" width="0.4064" layer="16"/>
+<wire x1="24" y1="55" x2="21.62" y2="55.84" width="0.4064" layer="16"/>
+<wire x1="41" y1="42" x2="42" y2="43" width="0.4064" layer="16"/>
+<wire x1="42" y1="43" x2="42" y2="47.19" width="0.4064" layer="16"/>
+<wire x1="25" y1="42" x2="41" y2="42" width="0.4064" layer="16"/>
 </signal>
 <signal name="N$32">
@@
 <contactref element="U$14" pad="D1"/>
 <contactref element="U$15" pad="D1"/>
-<wire x1="41" y1="28.19" x2="46.08920625" y2="28.19" width="0.4064" layer="16"/>
-<wire x1="41" y1="28.19" x2="37.08" y2="28.19" width="0.4064" layer="16"/>
+<wire x1="42" y1="28.19" x2="37.08" y2="28.19" width="0.4064" layer="16"/>
+<wire x1="42" y1="28.19" x2="46.08920625" y2="28.19" width="0.4064" layer="16"/>
 <wire x1="54.6631375" y1="28.19" x2="56.08" y2="28.19" width="0.4064" layer="16"/>
 <wire x1="51.7009375" y1="25.2278" x2="54.6631375" y2="28.19" width="0.4064" layer="16"/>
@@
 <wire x1="41" y1="41" x2="24" y2="41" width="0.4064" layer="16"/>
 <wire x1="24" y1="41" x2="23" y2="42" width="0.4064" layer="16"/>
-<wire x1="23" y1="42" x2="23" y2="51.92" width="0.4064" layer="16"/>
-<wire x1="42" y1="29.19" x2="41" y2="28.19" width="0.4064" layer="16"/>
-<wire x1="42" y1="40" x2="42" y2="29.19" width="0.4064" layer="16"/>
+<wire x1="23" y1="42" x2="23" y2="53" width="0.4064" layer="16"/>
 <contactref element="B1" pad="14"/>
-<wire x1="23" y1="51.92" x2="21.62" y2="53.3" width="0.4064" layer="16"/>
+<wire x1="23" y1="53" x2="21.62" y2="53.3" width="0.4064" layer="16"/>
+<wire x1="42" y1="40" x2="42" y2="28.19" width="0.4064" layer="16"/>
 </signal>
 <signal name="N$30">
@@
 <wire x1="106.05140625" y1="6.2278" x2="108.7009375" y2="6.2278" width="0.4064" layer="16"/>
 <contactref element="B1" pad="13"/>
-<wire x1="21.62" y1="50.76" x2="21.62" y2="6.38" width="0.4064" layer="16"/>
-<wire x1="21.62" y1="6.38" x2="23" y2="5" width="0.4064" layer="16"/>
+<wire x1="21.62" y1="50.76" x2="21.62" y2="41.38" width="0.4064" layer="16"/>
+<wire x1="21.62" y1="41.38" x2="23" y2="40" width="0.4064" layer="16"/>
+<wire x1="23" y1="40" x2="23" y2="5" width="0.4064" layer="16"/>
+<wire x1="23" y1="5" x2="24" y2="4" width="0.4064" layer="16"/>
 <wire x1="37" y1="9.11" x2="37.08" y2="9.19" width="0.4064" layer="16"/>
-<wire x1="37.81" y1="5" x2="42" y2="9.19" width="0.4064" layer="16"/>
-<wire x1="23" y1="5" x2="37.81" y2="5" width="0.4064" layer="16"/>
+<wire x1="41" y1="4" x2="42" y2="5" width="0.4064" layer="16"/>
+<wire x1="42" y1="5" x2="42" y2="9.19" width="0.4064" layer="16"/>
+<wire x1="24" y1="4" x2="41" y2="4" width="0.4064" layer="16"/>
 </signal>
 <signal name="N$26">
 <contactref element="S1" pad="1"/>
 <contactref element="B1" pad="23"/>
-<wire x1="9.5" y1="46.25" x2="9.5" y2="72.5" width="0.4064" layer="16"/>
+<wire x1="9.5" y1="43.25" x2="9.5" y2="72.5" width="0.4064" layer="16"/>
 <wire x1="9.5" y1="72.5" x2="13" y2="76" width="0.4064" layer="16"/>
 <wire x1="13" y1="76" x2="21.46" y2="76" width="0.4064" layer="16"/>
@@
 <wire x1="11" y1="48" x2="12" y2="47" width="0.4064" layer="16"/>
 <wire x1="12" y1="47" x2="14" y2="46.75" width="0.4064" layer="16"/>
-<wire x1="14" y1="46.75" x2="14.5" y2="46.25" width="0.4064" layer="16"/>
+<wire x1="14" y1="46.75" x2="14.5" y2="43.25" width="0.4064" layer="16"/>
 </signal>
 <signal name="N$29">
@@
 <wire x1="103.08920625" y1="66.19" x2="106.05140625" y2="63.2278" width="0.4064" layer="16"/>
 <wire x1="106.05140625" y1="63.2278" x2="108.7009375" y2="63.2278" width="0.4064" layer="16"/>
-<wire x1="21.62" y1="58.38" x2="34.19" y2="58.38" width="0.4064" layer="16"/>
-<wire x1="34.19" y1="58.38" x2="42" y2="66.19" width="0.4064" layer="16"/>
+<wire x1="21.62" y1="58.38" x2="23.38" y2="58.38" width="0.4064" layer="16"/>
+<wire x1="23.38" y1="58.38" x2="25" y2="60" width="0.4064" layer="16"/>
+<wire x1="25" y1="60" x2="41" y2="60" width="0.4064" layer="16"/>
+<wire x1="41" y1="60" x2="42" y2="61" width="0.4064" layer="16"/>
+<wire x1="42" y1="61" x2="42" y2="66.19" width="0.4064" layer="16"/>
 </signal>
 </signals>

Commit message: Final design; ordered
Parts:
- removed S1: RESET, SparkFun-Switches:TACTILE_SWITCH_PTH_12MM
- added RESET: RESET, SparkFun-Switches:TACTILE_SWITCH_PTH_12MM
- moved B1 6.40 mm to (9.00, 62.0)
- moved U$1 5.39 mm to (27.0, 68.0)
- moved U$10 5.39 mm to (103.0, 49.0)
- moved U$11 5.39 mm to (27.0, 30.0)
- moved U$12 5.39 mm to (46.0, 30.0)
- moved U$13 5.39 mm to (65.0, 30.0)
- moved U$14 5.39 mm to (84.0, 30.0)
- moved U$15 5.39 mm to (103.0, 30.0)
- moved U$16 5.39 mm to (27.0, 11.0)
- moved U$17 5.39 mm to (46.0, 11.0)
- moved U$18 5.39 mm to (65.0, 11.0)
- moved U$19 5.39 mm to (84.0, 11.0)
- moved U$2 5.39 mm to (46.0, 68.0)
- moved U$20 5.39 mm to (103.0, 11.0)
- moved U$3 5.39 mm to (65.0, 68.0)
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Connections:
- removed net N$28: B1.22, S1.3
- new net N$3: B1.23, RESET.3
- new net S$1: U$14.SW1, U$19.SW1, U$4.SW1, U$9.SW1
- new net S$2: U$10.SW1, U$15.SW1, U$20.SW1, U$5.SW1
- new net S$3: U$1.SW1, U$11.SW1, U$16.SW1, U$6.SW1
- net N$1: no longer U$1.SW1, U$11.SW1, U$16.SW1, U$6.SW1
- net N$26: now also B1.22, RESET.1; no longer B1.23, S1.1
- net N$4: no longer U$14.SW1, U$19.SW1, U$4.SW1, U$9.SW1
- net N$5: no longer U$10.SW1, U$15.SW1, U$20.SW1, U$5.SW1
Routing:
- net N$5: track 209.5 -> 146.8 mm
- net N$4: track 189.6 -> 127.0 mm
- net N$1: track 122.2 -> 61.5 mm
- net S$3: track 0.00 -> 58.7 mm
- net S$2: track 0.00 -> 58.7 mm
- net S$1: track 0.00 -> 58.7 mm
- net N$3: track 0.00 -> 49.1 mm
- net N$28: track 42.3 -> 0.00 mm
- net N$36: track 112.5 -> 117.5 mm
- net N$31: track 123.4 -> 128.1 mm
- net N$32: track 129.9 -> 134.5 mm
- net N$2: track 153.1 -> 149.1 mm
- net N$29: track 171.1 -> 167.1 mm
- net N$26: track 42.9 -> 46.8 mm
- net N$30: track 156.3 -> 158.6 mm
Other:
- board size 121 x 83 mm -> 112 x 79 mm
